File: mikoto.kicad_pcb (KiCad board)
At the start: 4 copper layers, 18 x 33.3 mm, 70 parts, among them J1 USB_C_Receptacle_USB2.0, J4 PTH, J5 PTH, U1 nRF52840, U2 BQ24075RGT, U3 XC6220B331MR, U4 mikoto-pins, U5 ESDR0502NMUTAG, Y1 32MHz, Y2 32.768 kHz

Commit message: paneling work.
Parts:
- added REF**: Tab, kikit:Tab, F.Cu at (9.50, 0.00)
- added REF**: Tab, kikit:Tab, F.Cu at (-9.50, 0.00)
